Commit message: Collision with spatula works, but spatula doesn't move yet.

File: zoom-chef/mmp_panda.urdf (robot description, URDF)
Before this commit: robot mmp_panda, 13 links, 12 joints
Links:
- link leftfinger: geometry collision mesh filename=../../../zoom-chef/panda/meshes/collision/finger.obj; visual mesh filename=../../../zoom-chef/panda/meshes/collision/finger.obj
- link rightfinger: geometry collision mesh filename=../../../zoom-chef/panda/meshes/collision/finger.obj; visual mesh filename=../../../zoom-chef/panda/meshes/collision/finger.obj

Commit message: The robot takes the imaginary burger from station1 to station2 and drops it on the imaginary grill.

File: zoom-chef/mmp_panda.urdf (robot description, URDF)
Before this commit: robot mmp_panda, 13 links, 12 joints
Links:
- link leftfinger: geometry collision mesh filename=../../../zoom-chef/panda/meshes/collision/finger.obj scale=1.5 1.0 2.5; visual mesh filename=../../../zoom-chef/panda/meshes/collision/finger.obj scale=1.5 1.0 2.5
- link rightfinger: geometry collision mesh filename=../../../zoom-chef/panda/meshes/collision/finger.obj scale=1.5 1.0 1.5; visual mesh filename=../../../zoom-chef/panda/meshes/collision/finger.obj scale=1.5 1.0 1.5

Commit message: burger collision mesh added

File: zoom-chef/mmp_panda.urdf (robot description, URDF)
Before this commit: robot mmp_panda, 13 links, 12 joints
Links:
- link leftfinger: mass 0.1 -> 1.0
- link rightfinger: mass 0.1 -> 1.0
Joints:
- joint finger_joint1: limit lower=0.0 upper=0.04 effort=20 velocity=0.2 -> lower=0.0 upper=0.04 effort=20 velocity=2
- joint finger_joint2: limit lower=0.0 upper=0.04 effort=20 velocity=0.2 -> lower=0.0 upper=0.04 effort=20 velocity=2

Commit message: The robot grabs the spatula, lifts the burger and puts it on the grill - NEW.

File: zoom-chef/mmp_panda.urdf (robot description, URDF)
Before this commit: robot mmp_panda, 13 links, 12 joints
Links:
- link leftfinger: mass 1.0 -> 1.5
- link rightfinger: mass 1.0 -> 1.5

Commit message: The robot puts the burger and buns on the grill.

File: zoom-chef/mmp_panda.urdf (robot description, URDF)
Before this commit: robot mmp_panda, 13 links, 12 joints
Links:
- link leftfinger: geometry collision mesh filename=../../../zoom-chef/panda/meshes/collision/finger.obj scale=5.0 1.0 2.5; visual mesh filename=../../../zoom-chef/panda/meshes/collision/finger.obj scale=5.0 1.0 2.5
- link rightfinger: geometry collision mesh filename=../../../zoom-chef/panda/meshes/collision/finger.obj scale=5.0 1.0 1.5; visual mesh filename=../../../zoom-chef/panda/meshes/collision/finger.obj scale=5.0 1.0 1.5

Commit message: Good boy made a burger

File: zoom-chef/mmp_panda.urdf (robot description, URDF)
Before this commit: robot mmp_panda, 13 links, 12 joints
Links:
- link link7: geometry collision mesh filename=../../../zoom-chef/panda/meshes/collision/hand.obj; visual mesh filename=../../../zoom-chef/panda/meshes/visual/chefhat.obj scale=0.01 0.01 0.01
